Commit message: IK modified dimensions and Hudson's control wishes

File: ArmControl/rsx_arm.urdf (robot description, URDF)
Before this commit: robot rsx_arm, 7 links, 6 joints
Links:
- link link2_shoulder: geometry visual box size=36 2 2
- link link3_elbow: geometry visual box size=32 2 2
Joints:
- joint joint2_elbow: origin xyz=36.5 0 0 rpy=0 0 0 -> xyz=36 0 0 rpy=0 0 0
- joint joint3_wrist1: origin xyz=33 0 0 rpy=0 1.5707963 0 -> xyz=32 0 0 rpy=0 1.5707963 0
