Commit message: standard orientations mode implemented + controls revised for a new arm + stability improvements

File: ArmControl/2018/rsx_arm.urdf (robot description, URDF)
Before this commit: robot rsx_arm, 7 links, 6 joints
Links:
- link link4_wrist1: geometry visual box size=4 3 2
- link link6_wrist3: geometry visual box size=4 3 2
